File: pcb/F407-v10/CanShark.sch (EAGLE design)
At the start: 86 parts, among them IC1 STM32F407V, IC2 KSZ8051MLL, K2 JACK_POWER_2,1, U1 SN65HVD230DR, U2 SN65HVD230DR, U3 LM2594M-ADJ, U4 LM2594M-ADJ

Commit message: Add JTAG/SWD and LEDs
Parts:
- added JP6: (no value), pinhead:PINHD-2X10
- added JP7: (no value), pinhead:PINHD-1X6
- added LED1, LED2: (no value), led:LEDSML0603
- added LED3, LED4, LED5: TLLG4400, led:TLLG4400
- added R36, R45, R46, R47: 10k, #Odpory:R-EU_R0603
- added R37, R38, R39, R40, R41: 100k, #Odpory:R-EU_R0603
- added R42: 0R, #Odpory:R-EU_R0603
- added R43: 1,2k, #Odpory:R-EU_R0603
- added R44: 330R, #Odpory:R-EU_R0603
Connections:
- new net JTG-TCK/SWCLK: JP6.9, R37.1
- new net JTG-TDI: JP6.5, R39.2
- new net JTG-TDO/SWO: JP6.13, R41.2
- new net JTG-TMS/SWDIO: JP6.7, R38.2
- new net JTG-TRST: JP6.3, R40.2
- new net LED_CAN1: LED3.C
- new net LED_CAN2: LED4.C
- new net LED_GLOBAL: LED5.C
- new net N$27: JP7.1, R42.2
- new net N$31: JP7.2
- new net N$32: JP7.4
- new net N$33: JP7.5
- new net N$34: JP7.6
- new net N$35: LED1.A, R43.1
- new net N$54: LED2.A, R44.1
- new net N$57: LED3.A, R45.1
- new net N$58: LED4.A, R46.1
- new net N$59: LED5.A, R47.1
- new net N$8: JP6.11, R36.1
- net +3V3: now also JP6.1, JP6.2, R38.1, R39.1, R40.1, R41.1, R42.1, R44.2, R45.2, R46.2, R47.2
- net GND: now also JP6.10, JP6.12, JP6.14, JP6.16, JP6.18, JP6.20, JP6.4, JP6.6, JP6.8, JP7.3, LED1.C, LED2.C, R36.2, R37.2
- net NRST: now also JP6.15
- net V+: now also R43.2

Commit message: add ADC
Parts:
- added C32, C33, C34, C37: 100nF, #Kondenzatory:KERAMICKYSMD0603
- added C35: 10nF, #Kondenzatory:KERAMICKYSMD0603
- added C36: 1uF, rcl:CPOL-EUSMCA
- added R48, R49: 0R, #Odpory:R-EU_R0603
- added R50: 200K, #Odpory:R-EU_R0603
- added R51, R53, R64: 100k, #Odpory:R-EU_R0603
- added R52, R58, R59, R63: 200k, #Odpory:R-EU_R0603
- added R54, R55, R56, R57: 10k, #Odpory:R-EU_R0603
- added R60: 22k, #Odpory:R-EU_R0603
- added R61: 11k, #Odpory:R-EU_R0603
- added R62: 300k, #Odpory:R-EU_R0603
- added U5: TSH24IDT, TSH24IDT:TSH24IDT
- added U6: MCP602-E/SN, MCP602:MCP602-E/SN
- R24, R25, R26, R28, R29, R31: value 4,7k -> 0R
Connections:
- removed net AIN1: IC1.PC0
- removed net AIN2: IC1.PA4
- removed net AIN3: IC1.PA5
- removed net AIN4: IC1.PA6
- removed net N$31: JP7.2
- removed net N$32: JP7.4
- removed net N$33: JP7.5
- removed net N$34: JP7.6
- new net ADC_CAN1DIFF: IC1.PC0, R63.2, R64.1
- new net ADC_CAN1H: IC1.PA5, R52.2, R53.1
- new net ADC_CAN1L: IC1.PA4, R50.2, R51.1
- new net ADC_TRIG: IC1.PA6, IC1.PC6, IC1.PE11, IC1.PE9, R58.2, R59.1
- new net ADC_TRIG_VALUE_PWM: IC1.PD12, R62.2
- new net CAN1L: JP2.2, R27.1, U1.CANL
- new net CANL: JP4.2, R32.1, U2.CANL
- new net N$60: R52.1, R56.1, U5.NEG_4, U5.OUT_4
- new net N$61: R50.1, R54.1, U5.NEG_3, U5.OUT_3
- new net N$62: R49.1, U5.POS_4
- new net N$63: R48.1, U5.POS_3
- new net N$64: R48.2
- new net N$65: R55.1, R63.1, U5.NEG_1, U5.OUT_2
- new net N$66: R54.2, R55.2, U5.NEG_2
- new net N$67: R56.2, R57.1, U5.POS_2
- new net N$68: R60.1, U5.POS_1, U6.VOUTA
- new net N$69: R58.1, U5.OUT_1
- new net N$70: R60.2, R61.1, U6.VINA-
- new net N$71: C34.1, R62.1, U6.VINA+
- net +3V3: now also C35.2, C36.+, C37.2
- net CAN1_MODE: now also IC1.PA8
- net CAN2_MODE: now also IC1.PC9
- net CAN2_RX: now also IC1.PB5; no longer IC1.PB6
- net CAN2_TX: now also IC1.PB6; no longer IC1.PB7
- net ETH_INTRP: now also IC1.PC8
- net ETH_RST: now also IC1.PC7
- net EXT_SUPPLY: no longer JP2.2, JP4.2, R27.1, R32.1, U1.CANL, U2.CANL
- net GND: now also C32.2, C33.2, C34.2, C35.1, C36.-, C37.1, R51.2, R53.2, R57.2, R59.2, R61.2, R64.2, U5.VCC-, U6.VSS
- net JTG-TCK/SWCLK: now also IC1.PA14, JP7.2
- net JTG-TDI: now also IC1.PA15
- net JTG-TDO/SWO: now also IC1.PB3, JP7.6
- net JTG-TMS/SWDIO: now also IC1.PA13, JP7.4
- net JTG-TRST: now also IC1.PB4
- net LED_CAN1: now also IC1.PD8
- net LED_CAN2: now also IC1.PD9
- net LED_GLOBAL: now also IC1.PD10
- net NRST: now also JP7.5
- net V+: now also C32.1, C33.1, U5.VCC+, U6.VDD
Other:
- moved on the sheet: C10, C9

Commit message: Add debug USART and split power supplies
Parts:
- added C38: (no value), rcl:CPOL-EUA/3216-18R
- added JP8: (no value), !pinhead:PINHD-1X4
Connections:
- removed net CAN1L: JP2.2, R27.1, U1.CANL
- removed net EXT_SUPPLY: C29.+, C30.+, K2.A, U3.VIN
- removed net N$11: JP2.3, JP3.2, U1.CANH
- removed net N$13: JP2.1
- removed net N$15: JP4.1
- removed net N$64: R48.2
- new net CAN1_H: JP2.3, JP3.2, R49.2, U1.CANH
- new net CAN1_L: JP2.2, R27.1, R48.2, U1.CANL
- new net EXTSUPPLY: C29.+, C30.+, C38.+, JP2.1, JP4.1, K2.A, U3.VIN, U4.VIN
- net +3V3: now also JP8.1
- net GND: now also C38.-, JP8.4
- net USART1_RX: now also JP8.3
- net USART1_TX: now also JP8.2
- net V+: no longer U4.VIN
Other:
- moved on the sheet: C27, C28, C29, C30, C31, C32, C33, C34, D1, D2, K2, L3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
